Commit message: test_modified

File: blue_arm_description/urdf/blue_arm.xacro (robot description, xacro)
@@ -444,3 +444,61 @@
       velocity="2.77" />
   </joint>
+  <link
+    name="suck_tool">
+    <inertial>
+      <origin
+        xyz="0 0 0"
+        rpy="0 0 0" />
+      <mass
+        value="0.08" />
+      <inertia
+        ixx="0.1"
+        ixy="0"
+        ixz="0"
+        iyy="0.1"
+        iyz="0"
+        izz="0.1" />
+    </inertial>
+    <visual>
+      <origin
+        xyz="0 0 0"
+        rpy="0 0 0" />
+      <geometry>
+        <mesh
+          filename="package://blue_arm_description/meshes/suck_model_3.STL" />
+      </geometry>
+      <material
+        name="">
+        <color
+          rgba="0.1 0.6 0.8 1" />
+      </material>
+    </visual>
+    <collision>
+      <origin
+        xyz="0 0 0"
+        rpy="0 0 0" />
+      <geometry>
+        <mesh
+          filename="package://blue_arm_description/meshes/suck_model_3.STL" />
+      </geometry>
+    </collision>
+  </link>
+  <joint
+    name="suck_tool_joint"
+    type="revolute">
+    <origin
+      xyz="0 -0.013 0.013"
+      rpy="0 1.57 0" />
+    <parent
+      link="link_7" />
+    <child
+      link="suck_tool" />
+    <axis
+      xyz="-1 0 0" />
+    <limit
+      lower="-3.1415926"
+      upper="3.1415926"
+      effort="1000"
+      velocity="2.77" />
+  </joint>
 </robot>

Commit message: before_reinstall_ubuntu

File: blue_arm_description/urdf/blue_arm.xacro (robot description, xacro)
@@ -486,5 +486,5 @@
   <joint
     name="suck_tool_joint"
-    type="revolute">
+    type="fixed">
     <origin
       xyz="0 -0.013 0.013"
@@ -496,9 +496,40 @@
     <axis
       xyz="-1 0 0" />
-    <limit
-      lower="-3.1415926"
-      upper="3.1415926"
-      effort="1000"
-      velocity="2.77" />
-  </joint>
+  </joint>
+  <!-- <link name = "pocker_place">
+    <visual>
+      <origin
+        xyz="0 0 0"
+        rpy="0 0 0" />
+      <geometry>
+        <mesh
+          filename="package://blue_arm_description/meshes/pocker_place_A1.STL" />
+      </geometry>
+      <material
+        name="">
+        <color
+          rgba="0.1 0.6 0.8 1" />
+      </material>
+    </visual>
+    <collision>
+      <origin
+        xyz="0 0 0"
+        rpy="0 0 0" />
+      <geometry>
+        <mesh
+          filename="package://blue_arm_description/meshes/pocker_place_A1.STL" />
+      </geometry>
+    </collision>
+  </link>
+  <joint
+    name="pocker_place_joint"
+    type="fixed">
+    <origin
+      xyz="0.38 -0.25 0.01"
+      rpy="2.03 0 1.6" />
+    <parent
+      link="world" />
+    <child
+      link="pocker_place" />
+  </joint> -->
 </robot>

File: blue_arm_description/urdf/bluearm_urdf_3.urdf (robot description, URDF)
Before this commit: robot bluearm_urdf_3, 8 links, 7 joints
Links:
- added link suck_tool, mass 6.3956; collision mesh filename=package://bluearm_urdf_3/meshes/suck_model.STL; visual mesh filename=package://bluearm_urdf_3/meshes/suck_model.STL
Joints:
- added joint suck_tool: type revolute, parent link_7, child suck_tool, origin xyz=0 0 0 rpy=0 0 0, axis 1 0 0, limit lower=0 upper=0 effort=0 velocity=0
